File: PiPico_OpenPLC.kicad_sch (KiCad schematic)
At the start: 13 parts, among them J10 Conn_01x03_Male, J11 Conn_01x03_Male, J9 Conn_01x06_Male, SW1 TS1187, U1 Pico, U3 LM4040DBZ-3

Commit message: snap
Parts:
- removed J9: Conn_01x06_Male, Connector_PinHeader_2.54mm:PinHeader_1x06_P2.54mm_Vertical, symbol Connector:Conn_01x06_Pin
- added C14 (x3): 50V 100nF X7R, Capacitor_SMD:C_0603_1608Metric, symbol Device:C
- added J14 (x2): 5 Pin 3.5mm, Connector_Phoenix_MC:PhoenixContact_MC_1,5_5-G-3.5_1x05_P3.50mm_Horizontal, symbol Connector_Generic:Conn_01x05
- added J16, J17, J18, J19, J20, J21: Conn_01x06_Male, Connector_PinHeader_2.54mm:PinHeader_1x06_P2.54mm_Vertical, symbol Connector:Conn_01x06_Pin
- added NT1 (x3): NetTie_2, NetTie:NetTie-2_SMD_Pad0.5mm, symbol Device:NetTie_2
- added U12, U15, U16: PCF8574, Package_SO:SOIC-16W_7.5x10.3mm_P1.27mm, symbol Interface_Expansion:PCF8574
Connections:
- net +3V3: now also J16.6 (Pin_6), J17.6 (Pin_6), J18.6 (Pin_6), J19.6 (Pin_6), NT1.2, NT1.2, NT1.2, U15.3 (A2), U16.1 (A0)
- net Di0: now also U15.4 (P0); no longer U1.9 (GPIO6)
- net Di1: now also U15.5 (P1); no longer U1.10 (GPIO7)
- net Di2: now also U15.6 (P2); no longer U1.11 (GPIO8)
- net Di3: now also U15.7 (P3); no longer U1.12 (GPIO9)
- net Di4: now also U15.9 (P4); no longer U1.14 (GPIO10)
- net Di5: now also U15.10 (P5); no longer U1.15 (GPIO11)
- net Di6: now also U15.11 (P6); no longer U1.16 (GPIO12)
- net Di7: now also U15.12 (P7); no longer U1.17 (GPIO13)
- net Do0: now also U12.4 (P0); no longer U1.19 (GPIO14)
- net Do1: now also U12.5 (P1); no longer U1.20 (GPIO15)
- net Do2: now also U12.6 (P2); no longer U1.21 (GPIO16)
- net Do3: now also U12.7 (P3); no longer U1.22 (GPIO17)
- net Do4: now also U12.9 (P4); no longer U1.24 (GPIO18)
- net Do5: now also U12.10 (P5); no longer U1.25 (GPIO19)
- net Do6: now also U12.11 (P6); no longer U1.26 (GPIO20)
- net Do7: now also U12.12 (P7); no longer U1.27 (GPIO21)
- net GND: now also C14.2, C14.2, C14.2, J16.1 (Pin_1), J17.1 (Pin_1), J18.1 (Pin_1), J19.1 (Pin_1), J20.6 (Pin_6), J21.6 (Pin_6), U12.1 (A0), U12.2 (A1), U12.3 (A2), U12.8 (VSS), U15.1 (A0), U15.2 (A1), U15.8 (VSS), U16.2 (A1), U16.3 (A2), U16.8 (VSS)
- net PWMo0: now also U1.26 (GPIO20); no longer U1.7 (GPIO5)
- net PWMo1: now also U1.27 (GPIO21); no longer U1.6 (GPIO4)
- net SCL / UART Rx / SPI ~{CS} renamed UART0_RX
- net UART0_RX: now also J17.4 (Pin_4)
- net SDA / UART Tx / SPI Rx renamed UART0_TX
- net UART0_TX: now also J17.5 (Pin_5)
- net SPI SCK renamed I2C1_SDA
- net I2C1_SDA: now also J18.3 (Pin_3)
- net SPI Tx renamed I2C1_SCL
- net I2C1_SCL: now also J18.2 (Pin_2)
- new net: C14.1, NT1.1, U16.16 (VDD)
- new net: C14.1, NT1.1, U15.16 (VDD)
- new net: J14.1 (Pin_1), J20.1 (Pin_1)
- new net: J14.2 (Pin_2), J20.2 (Pin_2)
- new net: J14.3 (Pin_3), J20.3 (Pin_3)
- new net: J14.4 (Pin_4), J20.4 (Pin_4)
- new net: J14.5 (Pin_5), J20.5 (Pin_5)
- new net: C14.1, NT1.1, U12.16 (VDD)
- new net: J14.1 (Pin_1), J21.1 (Pin_1)
- new net: J14.2 (Pin_2), J21.2 (Pin_2)
- new net: J14.3 (Pin_3), J21.3 (Pin_3)
- new net: J14.4 (Pin_4), J21.4 (Pin_4)
- new net: J14.5 (Pin_5), J21.5 (Pin_5)
- new net Do10: U16.6 (P2)
- new net Do11: U16.7 (P3)
- new net Do12: U16.9 (P4)
- new net Do13: U16.10 (P5)
- new net Do14: U16.11 (P6)
- new net Do15: U16.12 (P7)
- new net Do8: U16.4 (P0)
- new net Do9: U16.5 (P1)
- new net I2C0_SCL: J17.2 (Pin_2), U1.7 (GPIO5), U12.14 (SCL), U15.14 (SCL), U16.14 (SCL)
- new net I2C0_SDA: J17.3 (Pin_3), U1.6 (GPIO4), U12.15 (SDA), U15.15 (SDA), U16.15 (SDA)
- new net SPI0_CSn: J16.3 (Pin_3), U1.22 (GPIO17)
- new net SPI0_RX: J16.2 (Pin_2), U1.21 (GPIO16)
- new net SPI0_SCK: J16.4 (Pin_4), U1.24 (GPIO18)
- new net SPI0_TX: J16.5 (Pin_5), U1.25 (GPIO19)
- new net SPI1_CSn: J19.3 (Pin_3), U1.17 (GPIO13)
- new net SPI1_RX: J19.2 (Pin_2), U1.16 (GPIO12)
- new net SPI1_SCK: J19.4 (Pin_4), U1.19 (GPIO14)
- new net SPI1_TX: J19.5 (Pin_5), U1.20 (GPIO15)
- new net UART1_RX: J18.4 (Pin_4), U1.12 (GPIO9)
- new net UART1_TX: J18.5 (Pin_5), U1.11 (GPIO8)

Commit message: Preparation for future use.
Reworked to use i2c bus expanders.
added sketch for add-on boards.
Parts:
- added U13: PCF8574, Package_DFN_QFN:WQFN-16-1EP_3x3mm_P0.5mm_EP1.6x1.6mm, symbol Interface_Expansion:PCF8574
- added U14: ULN2803A, Package_DFN_QFN:QFN-20-1EP_4x4mm_P0.5mm_EP2.5x2.5mm, symbol Transistor_Array:ULN2803A
Other:
- sheet Digital_Output ports: added Do10, Do11, Do12, Do13, Do14, Do15, Do8, Do9; removed none

Commit message: Added Submodule, changed Ports to i2c
Parts:
- removed U13: PCF8574, Package_DFN_QFN:WQFN-16-1EP_3x3mm_P0.5mm_EP1.6x1.6mm, symbol Interface_Expansion:PCF8574
- removed U14: ULN2803A, Package_DFN_QFN:QFN-20-1EP_4x4mm_P0.5mm_EP2.5x2.5mm, symbol Transistor_Array:ULN2803A
- added HS1, HS2: Submodule, Project:Submodule, symbol Mechanical:Heatsink
Other:
- moved on the sheet: C14, F1, F2, F5, H1, H4, J10, J11, J14, J16, J17, J18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
